File: schema/iDLSchema/iDLSchema.kicad_sch (KiCad schematic)
At the start: 11 parts, among them U1 HC-SR04, U2 HC-SR04, U3 HC-SR04

Commit message: schema v0.2
Parts:
- removed R1, R3, R5: 330Ω, symbol Device:R_US
- removed R2, R4, R6: 470Ω, symbol Device:R_US
- added R1, R3, R5: 330Ω, Resistor_THT:R_Axial_DIN0207_L6.3mm_D2.5mm_P10.16mm_Horizontal, symbol 0_iDLSyms:R_US
- added R2, R4, R6: 470Ω, Resistor_THT:R_Axial_DIN0207_L6.3mm_D2.5mm_P10.16mm_Horizontal, symbol 0_iDLSyms:R_US
- MCU1: renamed from MCU?; footprint (none) -> 0_iDLFoot:Raspberry Pi Zero
- U1, U2, U3: footprint (none) -> 0_iDLFoot:HC-SR04
Connections:
- net +5V: now also U1.1 (VCC), U2.1 (VCC), U3.1 (VCC); no longer U1. (VCC), U2. (VCC), U3. (VCC)
- net GND: now also U1.4 (GND), U2.4 (GND), U3.4 (GND), R2.2, R4.1, R6.2; no longer U1. (VCC), U2. (VCC), U3. (VCC)
- net at MCU1.7 (GPIO4): now also R1.2, R2.1
- net at MCU1.11 (GPIO17): now also U1.2 (TRIG); no longer U1. (VCC)
- net at MCU1.13 (GPIO27): now also R3.1, R4.2
- net at MCU1.15 (GPIO22): now also U2.2 (TRIG); no longer U2. (VCC)
- net at MCU1.29 (GPIO5): now also R5.2, R6.1
- net at MCU1.31 (GPIO6): now also U3.2 (TRIG); no longer U3. (VCC)
- new net: R1.1, U1.3 (ECHO)
- new net: R3.2, U2.3 (ECHO)
- new net: R5.1, U3.3 (ECHO)

Commit message: schema v0.2
Parts:
- R1, R3, R5: value 330Ω -> 1kΩ
- R2, R4, R6: value 470Ω -> 2kΩ
Connections:
- net +5V: now also MCU1.4 (5V); no longer MCU1. (HDMI)
- net GND: now also MCU1.14 (GND), R2.1, R4.2; no longer MCU1. (HDMI), R2.2, R4.1
- net at MCU1. (HDMI): now also CAM1. (CAM)
- net at MCU1.11 (GPIO17): no longer U1.2 (TRIG)
- net at MCU1.12 (GPIO18): now also U1.2 (TRIG)
- net at MCU1.15 (GPIO22): no longer U2.2 (TRIG)
- net at MCU1.16 (GPIO23): now also R1.2, R2.2
- net at MCU1.18 (GPIO24): now also U2.2 (TRIG)
- net at MCU1.22 (GPIO25): now also R3.2, R4.1
- net at R5.2, R6.1: now also MCU1.36 (GPIO16); no longer MCU1.29 (GPIO5)
- net at MCU1.31 (GPIO6): no longer U3.2 (TRIG)
- net at MCU1.32 (GPIO12): now also U3.2 (TRIG)
- net at U2.3 (ECHO): now also R3.1; no longer R3.2
- now unconnected: MCU1.13 (GPIO27), MCU1.7 (GPIO4)
Other:
- moved on the sheet: CAM1, U1, U3
