File: schema/iDLSchema/iDLSchema.kicad_pcb (KiCad board)
At the start: 2 copper layers, 10 parts, among them U1 HC-SR04, U2 HC-SR04, U3 HC-SR04

Commit message: finished footprints
Parts:
- R1, R3, R5: value 330Ω -> 1kΩ
- R2, R4, R6: value 470Ω -> 2kΩ
- moved U2 314.6 mm to (386.1, 62.3), turned to 180 degrees
- moved R3 298.3 mm to (381.0, 75.0)
- moved R4 296.5 mm to (391.2, 83.8), turned to 180 degrees
- moved R6 172.9 mm to (250.2, 83.8), turned to 180 degrees
- moved U3 161.7 mm to (245.1, 62.3), turned to 180 degrees
- moved R5 147.3 mm to (240.0, 74.9)
- moved R2 58.2 mm to (99.1, 83.8)
- moved R1 50.4 mm to (99.1, 76.2)
- moved U1 43.7 mm to (104.1, 62.3), turned to 180 degrees
- moved MCU1 21.9 mm to (33.0, 96.5)
Connections:
- MCU1 pad 1: (no net) -> unconnected-(MCU1-Pad1)
- MCU1 pad 11: Net-(MCU1-Pad11) -> unconnected-(MCU1-Pad11)
- MCU1 pad 12: unconnected-(MCU1-Pad12) -> Net-(MCU1-Pad12)
- MCU1 pad 13: Net-(MCU1-Pad13) -> unconnected-(MCU1-Pad13)
- MCU1 pad 14: (no net) -> GND
- MCU1 pad 15: Net-(MCU1-Pad15) -> unconnected-(MCU1-Pad15)
- MCU1 pad 16: unconnected-(MCU1-Pad16) -> Net-(MCU1-Pad16)
- MCU1 pad 18: unconnected-(MCU1-Pad18) -> Net-(MCU1-Pad18)
- MCU1 pad 22: unconnected-(MCU1-Pad22) -> Net-(MCU1-Pad22)
- MCU1 pad 29: Net-(MCU1-Pad29) -> unconnected-(MCU1-Pad29)
- MCU1 pad 31: Net-(MCU1-Pad31) -> unconnected-(MCU1-Pad31)
- MCU1 pad 32: unconnected-(MCU1-Pad32) -> Net-(MCU1-Pad32)
- MCU1 pad 36: unconnected-(MCU1-Pad36) -> Net-(MCU1-Pad36)
- MCU1 pad 4: (no net) -> micro-USB
- MCU1 pad 7: Net-(MCU1-Pad7) -> unconnected-(MCU1-Pad7)
- R1 pad 2: Net-(MCU1-Pad7) -> Net-(MCU1-Pad16)
- R2 pad 1: Net-(MCU1-Pad7) -> GND
- R2 pad 2: GND -> Net-(MCU1-Pad16)
- R3 pad 1: Net-(MCU1-Pad13) -> Net-(R3-Pad1)
- R3 pad 2: Net-(R3-Pad2) -> Net-(MCU1-Pad22)
- R4 pad 1: GND -> Net-(MCU1-Pad22)
- R4 pad 2: Net-(MCU1-Pad13) -> GND
- R5 pad 2: Net-(MCU1-Pad29) -> Net-(MCU1-Pad36)
- R6 pad 1: Net-(MCU1-Pad29) -> Net-(MCU1-Pad36)
- U1 pad 2: Net-(MCU1-Pad11) -> Net-(MCU1-Pad12)
- U2 pad 2: Net-(MCU1-Pad15) -> Net-(MCU1-Pad18)
- U2 pad 3: Net-(R3-Pad2) -> Net-(R3-Pad1)
- U3 pad 2: Net-(MCU1-Pad31) -> Net-(MCU1-Pad32)
Routing:
- net micro-USB: track 0.00 -> 383.5 mm, vias 0 -> 6
- net Net-(MCU1-Pad22): track 0.00 -> 379.7 mm, vias 0 -> 2
- net Net-(MCU1-Pad18): track 0.00 -> 370.6 mm, vias 0 -> 2
- net Net-(MCU1-Pad36): track 0.00 -> 244.0 mm, vias 0 -> 1
- net Net-(MCU1-Pad32): track 0.00 -> 234.9 mm, vias 0 -> 2
- net Net-(MCU1-Pad16): track 0.00 -> 82.3 mm
- net Net-(MCU1-Pad12): track 0.00 -> 79.4 mm
- net Net-(R1-Pad1): track 0.00 -> 13.9 mm
- net Net-(R3-Pad1): track 0.00 -> 12.7 mm
- net Net-(R5-Pad1): track 0.00 -> 12.7 mm
- added copper zone on B.Cu, net GND
- added copper zone on F.Cu, net GND
Other:
- board outline added: 374.6 x 53.3 mm

Commit message: putting my name on it lol
Other:
- board text added: "Edited Oct 30, 2023"
- board text added: "Vrishak Vemuri | isDoorLocked PCB v0.3"
Changed lines of the file:
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@@
   )
   (gr_rect (start 30.48 45.72) (end 405.13 99.06) (layer "Edge.Cuts") (width 0.1) (fill none))
+  (gr_text "Vrishak Vemuri | isDoorLocked PCB v0.3\n" (at 339.09 93.98) (layer "F.Cu")
+    (effects (font (size 1.5 1.5) (thickness 0.3)))
+  )
+  (gr_text "Edited Oct 30, 2023\n" (at 386.08 93.98) (layer "F.Cu")
+    (effects (font (size 1.5 1.5) (thickness 0.3)))
+  )
   (segment (start 87.63 83.82) (end 35.56 83.82) (width 0.25) (layer "B.Cu") (net 8))
   (segment (start 101.6 69.85) (end 87.63 83.82) (width 0.25) (layer "B.Cu") (net 8))

Commit message: new labelling
Routing:
- net Net-(MCU1-Pad12): track 79.4 -> 80.2 mm
Other:
- board text added: "Edited Oct 31, 2023"
- board text removed: "Edited Oct 30, 2023"
Changed lines of the file:
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@@
   (title_block
     (title "iDLSchema_Footprint")
-    (date "2023-10-30")
-    (rev "0.3")
+    (date "2023-10-31")
+    (rev "0.3.1")
   )
   (layers
@@
     (property "Sheetname" "")
     (attr through_hole)
-    (fp_text reference "R6" (at 5.08 -2.37) (layer "F.SilkS")
-      (effects (font (size 1 1) (thickness 0.15)))
-    )
-    (fp_text value "2kΩ" (at 5.08 2.37) (layer "F.Fab")
+    (fp_text reference "R6" (at 13.97 0) (layer "F.SilkS")
+      (effects (font (size 1 1) (thickness 0.15)))
+    )
+    (fp_text value "2kΩ" (at -3.81 0) (layer "F.Fab")
       (effects (font (size 1 1) (thickness 0.15)))
     )
@@
     (property "Sheetname" "")
     (attr through_hole)
-    (fp_text reference "U1" (at 10.16 -5.08 180 unlocked) (layer "F.SilkS")
-      (effects (font (size 1 1) (thickness 0.15)))
-    )
-    (fp_text value "HC-SR04" (at 0 1 180 unlocked) (layer "F.Fab")
-      (effects (font (size 1 1) (thickness 0.15)))
-    )
-    (fp_text user "${REFERENCE}" (at 10.16 -7.62 180 unlocked) (layer "F.Fab")
+    (fp_text reference "U1" (at 10.16 -5.08 180 unlocked) (layer "F.SilkS") hide
+      (effects (font (size 1 1) (thickness 0.15)))
+    )
+    (fp_text value "HC-SR04" (at -10.16 2.571 180 unlocked) (layer "F.Fab")
+      (effects (font (size 1 1) (thickness 0.15)))
+    )
+    (fp_text user "${REFERENCE}" (at 10.16 -7.62 180 unlocked) (layer "F.Fab") hide
       (effects (font (size 1 1) (thickness 0.15)))
     )
@@
     (property "Sheetname" "")
     (attr through_hole)
-    (fp_text reference "R1" (at 5.08 -2.37) (layer "F.SilkS")
-      (effects (font (size 1 1) (thickness 0.15)))
-    )
-    (fp_text value "1kΩ" (at 5.08 2.37) (layer "F.Fab")
+    (fp_text reference "R1" (at -3.81 0) (layer "F.SilkS")
+      (effects (font (size 1 1) (thickness 0.15)))
+    )
+    (fp_text value "1kΩ" (at 13.97 0) (layer "F.Fab")
       (effects (font (size 1 1) (thickness 0.15)))
     )
@@
     (property "Sheetname" "")
     (attr through_hole)
-    (fp_text reference "U3" (at 10.16 -5.08 180 unlocked) (layer "F.SilkS")
-      (effects (font (size 1 1) (thickness 0.15)))
-    )
-    (fp_text value "HC-SR04" (at 0 1 180 unlocked) (layer "F.Fab")
-      (effects (font (size 1 1) (thickness 0.15)))
-    )
-    (fp_text user "${REFERENCE}" (at 10.16 -7.62 180 unlocked) (layer "F.Fab")
+    (fp_text reference "U3" (at 10.16 -5.08 180 unlocked) (layer "F.SilkS") hide
+      (effects (font (size 1 1) (thickness 0.15)))
+    )
+    (fp_text value "HC-SR04" (at -10.16 2.571 180 unlocked) (layer "F.Fab")
+      (effects (font (size 1 1) (thickness 0.15)))
+    )
+    (fp_text user "${REFERENCE}" (at 10.16 -7.62 180 unlocked) (layer "F.Fab") hide
       (effects (font (size 1 1) (thickness 0.15)))
     )
@@
     (property "Sheetname" "")
     (attr through_hole)
-    (fp_text reference "MCU1" (at 7.62 -48.26 unlocked) (layer "F.SilkS")
+    (fp_text reference "MCU1" (at 8.89 -48.26 unlocked) (layer "F.SilkS")
       (effects (font (size 1 1) (thickness 0.15)))
     )
@@
       (effects (font (size 1 1) (thickness 0.15)))
     )
-    (fp_text user "${REFERENCE}" (at 7.62 -45.72 unlocked) (layer "F.Fab")
+    (fp_text user "RPi Zero" (at 10.16 -45.72 unlocked) (layer "F.Fab")
       (effects (font (size 1 1) (thickness 0.15)))
     )
@@
     (property "Sheetname" "")
     (attr through_hole)
-    (fp_text reference "R5" (at 5.08 -2.37) (layer "F.SilkS")
-      (effects (font (size 1 1) (thickness 0.15)))
-    )
-    (fp_text value "1kΩ" (at 5.08 2.37) (layer "F.Fab")
+    (fp_text reference "R5" (at -3.81 0) (layer "F.SilkS")
+      (effects (font (size 1 1) (thickness 0.15)))
+    )
+    (fp_text value "1kΩ" (at 13.97 0) (layer "F.Fab")
       (effects (font (size 1 1) (thickness 0.15)))
     )
@@
     (property "Sheetname" "")
     (attr through_hole)
-    (fp_text reference "R4" (at 5.08 -2.37) (layer "F.SilkS")
-      (effects (font (size 1 1) (thickness 0.15)))
-    )
-    (fp_text value "2kΩ" (at 5.08 2.37) (layer "F.Fab")
+    (fp_text reference "R4" (at 13.97 0) (layer "F.SilkS")
+      (effects (font (size 1 1) (thickness 0.15)))
+    )
+    (fp_text value "2kΩ" (at -3.81 0) (layer "F.Fab")
       (effects (font (size 1 1) (thickness 0.15)))
     )
@@
     (property "Sheetname" "")
     (attr through_hole)
-    (fp_text reference "U2" (at 10.16 -5.08 180 unlocked) (layer "F.SilkS")
-      (effects (font (size 1 1) (thickness 0.15)))
-    )
-    (fp_text value "HC-SR04" (at 0 1 180 unlocked) (layer "F.Fab")
-      (effects (font (size 1 1) (thickness 0.15)))
-    )
-    (fp_text user "${REFERENCE}" (at 10.16 -7.62 180 unlocked) (layer "F.Fab")
+    (fp_text reference "U2" (at -3.81 -2.509 180 unlocked) (layer "F.SilkS") hide
+      (effects (font (size 1 1) (thickness 0.15)))
+    )
+    (fp_text value "HC-SR04" (at -10.16 2.571 180 unlocked) (layer "F.Fab")
+      (effects (font (size 1 1) (thickness 0.15)))
+    )
+    (fp_text user "${REFERENCE}" (at 10.16 -7.62 180 unlocked) (layer "F.Fab") hide
       (effects (font (size 1 1) (thickness 0.15)))
     )
@@
     (property "Sheetname" "")
     (attr through_hole)
-    (fp_text reference "R2" (at 5.08 -2.37) (layer "F.SilkS")
-      (effects (font (size 1 1) (thickness 0.15)))
-    )
-    (fp_text value "2kΩ" (at 5.08 2.37) (layer "F.Fab")
+    (fp_text reference "R2" (at -3.81 0) (layer "F.SilkS")
+      (effects (font (size 1 1) (thickness 0.15)))
+    )
+    (fp_text value "2kΩ" (at 13.97 0) (layer "F.Fab")
       (effects (font (size 1 1) (thickness 0.15)))
     )
@@
     (property "Sheetname" "")
     (attr through_hole)
-    (fp_text reference "R3" (at 5.08 -2.37) (layer "F.SilkS")
-      (effects (font (size 1 1) (thickness 0.15)))
-    )
-    (fp_text value "1kΩ" (at 5.08 2.37) (layer "F.Fab")
+    (fp_text reference "R3" (at -3.81 -0.02) (layer "F.SilkS")
+      (effects (font (size 1 1) (thickness 0.15)))
+    )
+    (fp_text value "1kΩ" (at 13.97 -0.02) (layer "F.Fab")
       (effects (font (size 1 1) (thickness 0.15)))
     )
@@
     (effects (font (size 1.5 1.5) (thickness 0.3)))
   )
-  (gr_text "Edited Oct 30, 2023\n" (at 386.08 93.98) (layer "F.Cu")
+  (gr_text "Edited Oct 31, 2023\n" (at 386.08 93.98) (layer "F.Cu")
     (effects (font (size 1.5 1.5) (thickness 0.3)))
   )
-  (segment (start 87.63 83.82) (end 35.56 83.82) (width 0.25) (layer "B.Cu") (net 8))
-  (segment (start 101.6 69.85) (end 87.63 83.82) (width 0.25) (layer "B.Cu") (net 8))
-  (segment (start 101.6 62.261) (end 101.6 69.85) (width 0.25) (layer "B.Cu") (net 8))
+  (segment (start 87.63 83.82) (end 91.44 80.01) (width 0.25) (layer "B.Cu") (net 8))
+  (segment (start 91.44 71.12) (end 96.52 66.04) (width 0.25) (layer "B.Cu") (net 8))
+  (segment (start 91.44 80.01) (end 91.44 71.12) (width 0.25) (layer "B.Cu") (net 8))
+  (segment (start 35.56 83.82) (end 87.63 83.82) (width 0.25) (layer "B.Cu") (net 8))
+  (segment (start 97.821 66.04) (end 101.6 62.261) (width 0.25) (layer "B.Cu") (net 8))
+  (segment (start 96.52 66.04) (end 97.821 66.04) (width 0.25) (layer "B.Cu") (net 8))
   (segment (start 109.22 78.74) (end 109.22 83.82) (width 0.25) (layer "F.Cu") (net 11))
   (segment (start 104.14 78.74) (end 106.68 76.2) (width 0.25) (layer "F.Cu") (net 11))
@@
   (segment (start 55.88 86.36) (end 66.04 96.52) (width 0.25) (layer "B.Cu") (net 14))
   (segment (start 45.72 76.2) (end 35.56 76.2) (width 0.25) (layer "B.Cu") (net 14))
-  (segment (start 391.16 74.95) (end 387.33 74.95) (width 0.25) (layer "F.Cu") (net 20))
-  (segment (start 134.62 91.44) (end 133.35 90.17) (width 0.25) (layer "F.Cu") (net 20))
+  (segment (start 389.87 74.95) (end 391.16 74.95) (width 0.25) (layer "F.Cu") (net 20))
+  (segment (start 374.65 78.74) (end 386.08 78.74) (width 0.25) (layer "F.Cu") (net 20))
   (segment (start 63.5 71.12) (end 35.56 71.12) (width 0.25) (layer "F.Cu") (net 20))
-  (segment (start 256.54 91.44) (end 134.62 91.44) (width 0.25) (layer "F.Cu") (net 20))
-  (segment (start 383.54 78.74) (end 377.335 84.945) (width 0.25) (layer "F.Cu") (net 20))
   (segment (start 66.04 73.66) (end 63.5 71.12) (width 0.25) (layer "F.Cu") (net 20))
-  (segment (start 377.335 84.945) (end 263.035 84.945) (width 0.25) (layer "F.Cu") (net 20))
-  (segment (start 387.33 74.95) (end 383.54 78.74) (width 0.25) (layer "F.Cu") (net 20))
-  (segment (start 263.035 84.945) (end 256.54 91.44) (width 0.25) (layer "F.Cu") (net 20))
-  (segment (start 86.36 90.17) (end 77.47 81.28) (width 0.25) (layer "F.Cu") (net 20))
-  (segment (start 133.35 90.17) (end 86.36 90.17) (width 0.25) (layer "F.Cu") (net 20))
+  (segment (start 133.35 90.17) (end 134.62 91.44) (width 0.25) (layer "F.Cu") (net 20))
+  (segment (start 77.47 81.28) (end 86.36 90.17) (width 0.25) (layer "F.Cu") (net 20))
+  (segment (start 361.95 91.44) (end 374.65 78.74) (width 0.25) (layer "F.Cu") (net 20))
+  (segment (start 134.62 91.44) (end 361.95 91.44) (width 0.25) (layer "F.Cu") (net 20))
+  (segment (start 86.36 90.17) (end 133.35 90.17) (width 0.25) (layer "F.Cu") (net 20))
   (segment (start 391.16 83.82) (end 391.16 74.95) (width 0.25) (layer "F.Cu") (net 20))
+  (segment (start 386.08 78.74) (end 389.87 74.95) (width 0.25) (layer "F.Cu") (net 20))
   (via (at 77.47 81.28) (size 0.8) (drill 0.4) (layers "F.Cu" "B.Cu") (net 20))
   (via (at 66.04 73.66) (size 0.8) (drill 0.4) (layers "F.Cu" "B.Cu") (net 20))

Commit message: layer rev, need to put a ne t
Parts:
- RPi Zero: renamed from MCU1
Routing:
- removed copper zone on B.Cu, net GND
- removed copper zone on F.Cu, net GND
Changed lines of the file:
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@@
     (title "iDLSchema_Footprint")
     (date "2023-10-31")
-    (rev "0.3.1")
+    (rev "0.3.2")
   )
   (layers
@@
       (layerselection 0x00010fc_ffffffff)
       (disableapertmacros false)
-      (usegerberextensions false)
-      (usegerberattributes true)
-      (usegerberadvancedattributes true)
-      (creategerberjobfile true)
+      (usegerberextensions true)
+      (usegerberattributes false)
+      (usegerberadvancedattributes false)
+      (creategerberjobfile false)
       (svguseinch false)
       (svgprecision 6)
@@
       (psa4output false)
       (plotreference true)
-      (plotvalue true)
+      (plotvalue false)
       (plotinvisibletext false)
       (sketchpadsonfab false)
-      (subtractmaskfromsilk false)
+      (subtractmaskfromsilk true)
       (outputformat 1)
       (mirror false)
-      (drillshape 1)
+      (drillshape 0)
       (scaleselection 1)
-      (outputdirectory "")
+      (outputdirectory "drill/")
     )
   )
@@
       (effects (font (size 1 1) (thickness 0.15)))
     )
-    (fp_text value "2kΩ" (at -3.81 0) (layer "F.Fab")
+    (fp_text value "2kΩ" (at -3.81 0) (layer "F.SilkS")
       (effects (font (size 1 1) (thickness 0.15)))
     )
@@
       (effects (font (size 1 1) (thickness 0.15)))
     )
-    (fp_text value "HC-SR04" (at -10.16 2.571 180 unlocked) (layer "F.Fab")
+    (fp_text value "HC-SR04" (at -10.16 2.571 180 unlocked) (layer "F.SilkS")
       (effects (font (size 1 1) (thickness 0.15)))
     )
@@
       (effects (font (size 1 1) (thickness 0.15)))
     )
-    (fp_text value "1kΩ" (at 13.97 0) (layer "F.Fab")
+    (fp_text value "1kΩ" (at 13.97 0) (layer "F.SilkS")
       (effects (font (size 1 1) (thickness 0.15)))
     )
@@
       (effects (font (size 1 1) (thickness 0.15)))
     )
-    (fp_text value "HC-SR04" (at -10.16 2.571 180 unlocked) (layer "F.Fab")
+    (fp_text value "HC-SR04" (at -10.16 2.571 180 unlocked) (layer "F.SilkS")
       (effects (font (size 1 1) (thickness 0.15)))
     )
@@
     (property "Sheetname" "")
     (attr through_hole)
-    (fp_text reference "MCU1" (at 8.89 -48.26 unlocked) (layer "F.SilkS")
-      (effects (font (size 1 1) (thickness 0.15)))
-    )
-    (fp_text value "Raspberry_Pi_Zero_W" (at 0 7.62 unlocked) (layer "F.Fab")
+    (fp_text reference "RPi Zero" (at 10.16 -48.26 unlocked) (layer "F.SilkS")
+      (effects (font (size 1 1) (thickness 0.15)))
+    )
+    (fp_text value "Raspberry_Pi_Zero_W" (at 0 7.62 unlocked) (layer "F.Fab") hide
       (effects (font (size 1 1) (thickness 0.15)))
     )
@@
       (effects (font (size 1 1) (thickness 0.15)))
     )
-    (fp_text value "1kΩ" (at 13.97 0) (layer "F.Fab")
+    (fp_text value "1kΩ" (at 13.97 0) (layer "F.SilkS")
       (effects (font (size 1 1) (thickness 0.15)))
     )
@@
       (effects (font (size 1 1) (thickness 0.15)))
     )
-    (fp_text value "2kΩ" (at -3.81 0) (layer "F.Fab")
+    (fp_text value "2kΩ" (at -3.81 0) (layer "F.SilkS")
       (effects (font (size 1 1) (thickness 0.15)))
     )
@@
       (effects (font (size 1 1) (thickness 0.15)))
     )
-    (fp_text value "HC-SR04" (at -10.16 2.571 180 unlocked) (layer "F.Fab")
+    (fp_text value "HC-SR04" (at -10.16 2.571 180 unlocked) (layer "F.SilkS")
       (effects (font (size 1 1) (thickness 0.15)))
     )
@@
       (effects (font (size 1 1) (thickness 0.15)))
     )
-    (fp_text value "2kΩ" (at 13.97 0) (layer "F.Fab")
+    (fp_text value "2kΩ" (at 13.97 0) (layer "F.SilkS")
       (effects (font (size 1 1) (thickness 0.15)))
     )
@@
       (effects (font (size 1 1) (thickness 0.15)))
     )
-    (fp_text value "1kΩ" (at 13.97 -0.02) (layer "F.Fab")
+    (fp_text value "1kΩ" (at 13.97 -0.02) (layer "F.SilkS")
       (effects (font (size 1 1) (thickness 0.15)))
     )
@@
   )
   (gr_rect (start 30.48 45.72) (end 405.13 99.06) (layer "Edge.Cuts") (width 0.1) (fill none))
-  (gr_text "Vrishak Vemuri | isDoorLocked PCB v0.3\n" (at 339.09 93.98) (layer "F.Cu")
+  (gr_text "Vrishak Vemuri | isDoorLocked PCB v0.3\n" (at 339.09 93.98) (layer "F.SilkS")
     (effects (font (size 1.5 1.5) (thickness 0.3)))
   )
-  (gr_text "Edited Oct 31, 2023\n" (at 386.08 93.98) (layer "F.Cu")
+  (gr_text "Edited Oct 31, 2023\n" (at 386.08 93.98) (layer "F.SilkS")
     (effects (font (size 1.5 1.5) (thickness 0.3)))
   )
@@
   (segment (start 245.079 62.261) (end 245.11 62.261) (width 0.25) (layer "B.Cu") (net 33))
   (segment (start 381 74.95) (end 381 62.261) (width 0.25) (layer "F.Cu") (net 34))
-  (zone (net 30) (net_name "GND") (layer "F.Cu") (hatch edge 0.508)
-    (connect_pads (clearance 0.508))
-    (min_thickness 0.254) (filled_areas_thickness no)
-    (fill yes (thermal_gap 0.508) (thermal_bridge_width 0.508))
-    (polygon
-      (pts
-        (xy 405.13 99.06)
-        (xy 30.48 99.06)
-        (xy 30.48 45.72)
-        (xy 405.13 45.72)
-      )
-    )
-  )
-  (zone (net 30) (net_name "GND") (layer "B.Cu") (hatch edge 0.508)
-    (connect_pads (clearance 0.508))
-    (min_thickness 0.254) (filled_areas_thickness no)
-    (fill yes (thermal_gap 0.508) (thermal_bridge_width 0.508))
-    (polygon
-      (pts
-        (xy 405.13 99.06)
-        (xy 30.48 99.06)
-        (xy 30.48 45.72)
-        (xy 405.13 45.72)
-      )
-    )
-  )
 )

Commit message: new gerbers
Routing:
- added copper zone on B.Cu, net GND
- added copper zone on F.Cu, net GND
Other:
- board text added: "Vrishak Vemuri | isDoorLocked PCB v0.3.2"
- board text removed: "Vrishak Vemuri | isDoorLocked PCB v0.3"
Changed lines of the file:
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@@
       (drillshape 0)
       (scaleselection 1)
-      (outputdirectory "drill/")
+      (outputdirectory "gerber/")
     )
   )
@@
   )
   (gr_rect (start 30.48 45.72) (end 405.13 99.06) (layer "Edge.Cuts") (width 0.1) (fill none))
-  (gr_text "Vrishak Vemuri | isDoorLocked PCB v0.3\n" (at 339.09 93.98) (layer "F.SilkS")
+  (gr_text "Vrishak Vemuri | isDoorLocked PCB v0.3.2\n" (at 339.09 93.98) (layer "F.SilkS")
     (effects (font (size 1.5 1.5) (thickness 0.3)))
   )
@@
   (segment (start 245.079 62.261) (end 245.11 62.261) (width 0.25) (layer "B.Cu") (net 33))
   (segment (start 381 74.95) (end 381 62.261) (width 0.25) (layer "F.Cu") (net 34))
+  (zone (net 30) (net_name "GND") (layer "F.Cu") (hatch edge 0.508)
+    (connect_pads (clearance 0.508))
+    (min_thickness 0.254) (filled_areas_thickness no)
+    (fill yes (thermal_gap 0.508) (thermal_bridge_width 0.508))
+    (polygon
+      (pts
+        (xy 405.13 99.06)
+        (xy 30.48 99.06)
+        (xy 30.48 45.72)
+        (xy 405.13 45.72)
+      )
+    )
+  )
+  (zone (net 30) (net_name "GND") (layer "B.Cu") (hatch edge 0.508)
+    (connect_pads (clearance 0.508))
+    (min_thickness 0.254) (filled_areas_thickness no)
+    (fill yes (thermal_gap 0.508) (thermal_bridge_width 0.508))
+    (polygon
+      (pts
+        (xy 405.13 99.06)
+        (xy 30.48 99.06)
+        (xy 30.48 45.72)
+        (xy 405.13 45.72)
+      )
+    )
+  )
 )
